Commit message: fix base and world frame mismatch

File: robots/common/franka_robot.xacro (robot description, xacro)
@@ -96,12 +96,20 @@
       <xacro:if value="${parent != ''}">
         <!-- Gazebo requires a joint to a link called "world" for statically mounted robots -->
-        <xacro:if value="${parent == 'world'}">
-          <link name="${parent}" />
-        </xacro:if>
-        <joint name="${parent}_joint" type="fixed">
+        <link name="${parent}" />
+        <!-- <joint name="${parent}_joint" type="fixed">
           <origin xyz="${xyz}" rpy="${rpy}" />
           <parent link="${parent}" />
           <child  link="${arm_prefix}${arm_id}_link0" />
-        </joint>
+        </joint> -->
+      <link name="base"/>
+      <joint name="world_to_base" type="fixed">
+        <parent link="world"/>
+        <child link="base"/>
+      </joint>
+      <joint name="${parent}_joint" type="fixed">
+        <origin xyz="${xyz}" rpy="${rpy}" />
+        <parent link="${parent}" />
+        <child  link="${arm_prefix}${arm_id}_link0" />
+      </joint>
       </xacro:if>
       <xacro:gazebo-joint joint="${arm_prefix}${arm_id}_joint1" transmission="hardware_interface/PositionJointInterface" />

Commit message: merge branch add-camera

File: robots/common/franka_robot.xacro (robot description, xacro)
@@ -28,4 +28,5 @@
                       arm_prefix:=''
                       description_pkg:='franka_description'
+                      use_camera:='true'
                       connected_to:='base'">
     <xacro:include filename="$(find franka_description)/robots/common/utils.xacro" />
@@ -54,4 +55,8 @@
       <xacro:if value="${arm_id == 'fr3' or arm_id == 'fer' or arm_id == 'fr3v2'}">
         <xacro:property name="ee_color" value="white" />
+      </xacro:if>
+      <xacro:property name="xyz_ee" value="0.0 0.0 0.0"/>
+      <xacro:if value="${use_camera}">
+        <xacro:property name="xyz_ee" value="0.0 0.0 0.05505"/>
       </xacro:if>
       <xacro:property name="connection" value="${special_connection if special_connection != '' else arm_id + '_link8'}" />
@@ -147,4 +152,10 @@
       </xacro:if>
     </xacro:if>
+    <xacro:if value="${use_camera}">
+      <xacro:include filename="$(find realsense2_description)/urdf/_d435.urdf.xacro"/>
+      <xacro:sensor_d435 name="camera" parent="${arm_prefix}${arm_id}_link8">
+        <origin xyz="0 0 0" rpy="0 0 0"/>
+      </xacro:sensor_d435>
+    </xacro:if>
     <xacro:if value="${ros2_control}">
       <xacro:include filename="$(find franka_description)/robots/common/franka_arm.ros2_control.xacro"/>

File: robots/fr3/fr3.srdf.xacro (robot description, xacro)
@@ -7,6 +7,4 @@
     This argument is ignored.
   -->
-  <xacro:arg name="arm_id" default="fr3" />
-  <!-- The prefix of the robot -->
   <xacro:arg name="arm_prefix" default="" />
   <!-- Don't print a prefix for joints, visuals, and links? -->
@@ -16,9 +14,11 @@
   <!-- Which end-effector would be mounted at the flange?" -->
   <xacro:arg name="ee_id" default="franka_hand" />
+  <xacro:arg name="camera" default="true" />
   <xacro:franka_arm_srdf arm_id="$(arg arm_id)"
                       hand="$(arg hand)"
                       ee_id="$(arg ee_id)"
                       no_prefix="$(arg no_prefix)"
-                      arm_prefix= "$(arg arm_prefix)">
+                      arm_prefix= "$(arg arm_prefix)"
+                      camera="$(arg camera)">
   </xacro:franka_arm_srdf>
 </robot>

File: robots/fr3/fr3.urdf.xacro (robot description, xacro)
@@ -2,4 +2,5 @@
 <robot xmlns:xacro="http://www.ros.org/wiki/xacro" name="fr3">
   <xacro:include filename="$(find franka_description)/robots/common/franka_robot.xacro"/>
+  <xacro:include filename="$(find realsense2_description)/urdf/_d435.urdf.xacro"/>
   <!--
     DEPRECATION NOTICE
@@ -44,4 +45,6 @@
   <!-- Name of the description package -->
   <xacro:arg name="description_pkg" default="franka_description" />
+  <!-- Use the D435 camera or not -->
+  <xacro:arg name="use_camera" default="true" />
   <!-- Append an underscore to the user-provided prefix, if non-empty. -->
   <xacro:property name="prefix" value="$(arg arm_prefix)"/>
@@ -70,4 +73,5 @@
                       arm_prefix="${modified_prefix}"
                       description_pkg="$(arg description_pkg)"
+                      use_camera="$(arg use_camera)"
                       connected_to= "base">
   </xacro:franka_robot>
