Commit message: test

File: robots/common/franka_arm.ros2_control.xacro (robot description, xacro)
@@ -52,7 +52,7 @@
       </xacro:macro>
       <xacro:configure_joint joint_name="${arm_prefix}${arm_id}_joint1" initial_position="0.0"/>
-      <xacro:configure_joint joint_name="${arm_prefix}${arm_id}_joint2" initial_position="${-pi/4}"/>
+      <xacro:configure_joint joint_name="${arm_prefix}${arm_id}_joint2" initial_position="0.0"/>
       <xacro:configure_joint joint_name="${arm_prefix}${arm_id}_joint3" initial_position="0.0"/>
-      <xacro:configure_joint joint_name="${arm_prefix}${arm_id}_joint4" initial_position="${-3*pi/4}"/>
+      <xacro:configure_joint joint_name="${arm_prefix}${arm_id}_joint4" initial_position="-0.1"/>
       <xacro:configure_joint joint_name="${arm_prefix}${arm_id}_joint5" initial_position="0.0"/>
       <xacro:configure_joint joint_name="${arm_prefix}${arm_id}_joint6" initial_position="${pi/2}"/>

File: robots/common/franka_robot.xacro (robot description, xacro)
@@ -32,4 +32,5 @@
     <xacro:include filename="$(find franka_description)/robots/common/utils.xacro" />
     <xacro:include filename="$(find franka_description)/robots/common/franka_arm.xacro" />
+    <xacro:include filename="$(find franka_description)/robots/common/_d435.urdf.xacro" />
     <xacro:franka_arm
       arm_id="${arm_id}"
@@ -153,9 +154,15 @@
     </xacro:if>
     <xacro:if value="${use_camera}">
-      <xacro:include filename="$(find realsense2_description)/urdf/_d435.urdf.xacro"/>
+      <xacro:include filename="$(find franka_description)/robots/common/_d435.urdf.xacro"/>
       <xacro:sensor_d435 name="camera" parent="${arm_prefix}${arm_id}_link8">
         <origin xyz="0 0 0" rpy="0 0 0"/>
       </xacro:sensor_d435>
     </xacro:if>
+    <!-- <xacro:if value="${use_camera}">
+      <xacro:include filename="$(find realsense_gazebo_plugin)/xacro/depthcam.xacro"/>
+      <xacro:realsense_d435 sensor_name="d435" parent_link="${arm_prefix}${arm_id}_link8" rate="10">
+        <origin rpy="0 0 0 " xyz="0 0 0"/>
+      </xacro:realsense_d435>
+    </xacro:if> -->
     <xacro:if value="${ros2_control}">
       <xacro:include filename="$(find franka_description)/robots/common/franka_arm.ros2_control.xacro"/>

File: robots/fr3/fr3.urdf.xacro (robot description, xacro)
@@ -2,5 +2,5 @@
 <robot xmlns:xacro="http://www.ros.org/wiki/xacro" name="fr3">
   <xacro:include filename="$(find franka_description)/robots/common/franka_robot.xacro"/>
-  <xacro:include filename="$(find realsense2_description)/urdf/_d435.urdf.xacro"/>
+  <xacro:include filename="$(find franka_description)/robots/common/_d435.urdf.xacro"/>
   <!--
     DEPRECATION NOTICE
