Commit message: increase max gripper width

File: end_effectors/common/franka_hand.xacro (robot description, xacro)
@@ -117,5 +117,5 @@
       <origin xyz="0 0 0.0584" rpy="0 0 0" />
       <axis xyz="0 1 0" />
-      <limit effort="100" lower="0.0" upper="0.04" velocity="0.2" />
+      <limit effort="100" lower="0.0" upper="0.05" velocity="0.2" />
       <dynamics damping="0.3" />
     </joint>
@@ -125,5 +125,5 @@
       <origin xyz="0 0 0.0584" rpy="0 0 ${pi}" />
       <axis xyz="0 1 0" />
-      <limit effort="100" lower="0.0" upper="0.04" velocity="0.2" />
+      <limit effort="100" lower="0.0" upper="0.05" velocity="0.2" />
       <mimic joint="${ee_prefix}finger_joint1" />
       <dynamics damping="0.3" />

File: end_effectors/franka_hand/franka_hand.srdf.xacro (robot description, xacro)
@@ -10,5 +10,5 @@
     </group>
     <group_state name="open" group="${prefix}hand">
-      <joint name="${prefix}finger_joint1" value="0.03"/>
+      <joint name="${prefix}finger_joint1" value="0.05"/>
       <!-- <joint name="${prefix}finger_joint2" value="0.03"/> -->
     </group_state>
